Commit message: 第四次提交 完成了深度相机节点的配置

File: src/lerobot/description_lerobot/urdf/lerobot_camera.urdf (robot description, URDF)
Before this commit: robot so_arm_100_5dof, 9 links, 8 joints
Links:
- added link depth_camera, mass 0.01; collision box size=0.02 0.10 0.02; visual box size=0.02 0.10 0.02
Joints:
- added joint depth_camera: type fixed, parent base_link, child depth_camera, origin xyz=0 -1 0.5 rpy=0 0.5 1.57

File: src/lerobot/description_lerobot/urdf/rviz_lerobot_camera.urdf (robot description, URDF)
Before this commit: robot so_arm_100_5dof, 11 links, 10 joints
Links:
- removed link depth_camera_link
- removed link world
- added link depth_camera, mass 0.01; collision box size=0.02 0.10 0.02; visual box size=0.02 0.10 0.02
- link Base: geometry collision mesh filename=package://description_lerobot/models/so_arm_100_5dof/meshes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 scale=0.9 0.9 0.9; visual mesh filename=package://description_lerobot/models/so_arm_100_5dof/meshes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
- link End_Effector: geometry visual box size=0.01 0.01 0.01
- link Fixed_Gripper: geometry collision mesh filename=package://description_lerobot/models/so_arm_100_5dof/meshes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 scale=0.9 0.9 0.9; visual mesh filename=package://description_lerobot/models/so_arm_100_5dof/meshes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
- link Lower_Arm: geometry collision mesh filename=package://description_lerobot/models/so_arm_100_5dof/meshes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 scale=0.9 0.9 0.9; visual mesh filename=package://description_lerobot/models/so_arm_100_5dof/meshes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
- link Moving_Jaw: geometry collision mesh filename=package://description_lerobot/models/so_arm_100_5dof/meshes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 scale=0.9 0.9 0.9; visual mesh filename=package://description_lerobot/models/so_arm_100_5dof/meshes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
- link Shoulder_Rotation_Pitch: geometry collision mesh filename=package://description_lerobot/models/so_arm_100_5dof/meshes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 scale=0.9 0.9 0.9; visual mesh filename=package://description_lerobot/models/so_arm_100_5dof/meshes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
- link Upper_Arm: geometry collision mesh filename=package://description_lerobot/models/so_arm_100_5dof/meshes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 scale=0.9 0.9 0.9; visual mesh filename=package://description_lerobot/models/so_arm_100_5dof/meshes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
- link Wrist_Pitch_Roll: geometry collision mesh filename=package://description_lerobot/models/so_arm_100_5dof/meshes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 scale=0.9 0.9 0.9; visual mesh filename=package://description_lerobot/models/so_arm_100_5dof/meshes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
- link base_link: mass 0.1 -> None; geometry 
Joints:
- removed joint depth_camera_fixed_joint
- removed joint fixed
- added joint depth_camera: type fixed, parent base_link, child depth_camera, origin xyz=0 -1 0.5 rpy=0 0.5 1.57
- joint Elbow: parent base_link -> Upper_Arm
- joint End_Effector_Joint: parent base_link -> Fixed_Gripper
- joint Gripper: parent base_link -> Fixed_Gripper
- joint Shoulder_Pitch: parent base_link -> Shoulder_Rotation_Pitch
- joint Shoulder_Rotation: parent base_link -> Base
- joint Wrist_Pitch: parent base_link -> Lower_Arm
- joint Wrist_Roll: parent base_link -> Wrist_Pitch_Roll
- joint base_link_joint: origin xyz=0 0 0.2 rpy=0 0 0 -> xyz=0 0 0 rpy=0 0 0
